Commit message: Add analyze file and and sensor function

File: body.urdf (robot description, URDF)
Before this commit: robot robot, 3 links, 2 joints
Links:
- removed link backleg
- removed link frontleg
- removed link torso
- added link BackLeg, mass 1; collision box size=1 1 1; visual box size=1 1 1
- added link FrontLeg, mass 1; collision box size=1 1 1; visual box size=1 1 1
- added link Torso, mass 1; collision box size=1 1 1; visual box size=1 1 1
Joints:
- removed joint torso_backleg
- removed joint torso_frontleg
- added joint Torso_BackLeg: type revolute, parent Torso, child BackLeg, origin xyz=1 0 1 rpy=0 0 0, axis 0 1 0, limit lower=-3.14159 upper=3.14159 effort=0.0 velocity=0.0
- added joint Torso_FrontLeg: type revolute, parent Torso, child FrontLeg, origin xyz=2 0 1 rpy=0 0 0, axis 0 1 0, limit lower=-3.14159 upper=3.14159 effort=0.0 velocity=0.0

Commit message: simulation crash for hexaped

File: body.urdf (robot description, URDF)
Before this commit: robot robot, 9 links, 8 joints
Links:
- removed link BackLeg
- removed link BackLowerLeg
- removed link FrontLeg
- removed link FrontLowerLeg
- removed link LeftLeg
- removed link LeftLowerLeg
- removed link RightLeg
- removed link RightLowerLeg
- added link LeftLeg1, mass 1; collision box size=0.2 1 0.2; visual box size=0.2 1 0.2
- added link LeftLeg3, mass 1; collision box size=0.2 1 0.2; visual box size=0.2 1 0.2
- added link LeftLowerLeg1, mass 1; collision box size=0.2 0.2 1; visual box size=0.2 0.2 1
- added link LeftLowerLeg3, mass 1; collision box size=0.2 0.2 1; visual box size=0.2 0.2 1
- added link RightLeg1, mass 1; collision box size=0.2 1 0.2; visual box size=0.2 1 0.2
- added link RightLeg3, mass 1; collision box size=0.2 1 0.2; visual box size=0.2 1 0.2
- added link RightLowerLeg1, mass 1; collision box size=0.2 0.2 1; visual box size=0.2 0.2 1
- added link RightLowerLeg3, mass 1; collision box size=0.2 0.2 1; visual box size=0.2 0.2 1
- link Torso: geometry collision box size=2 1 1; visual box size=2 1 1
Joints:
- removed joint BackLeg_BackLowerLeg
- removed joint FrontLeg_FrontLowerLeg
- removed joint LeftLeg_LeftLowerLeg
- removed joint RightLeg_RightLowerLeg
- removed joint Torso_BackLeg
- removed joint Torso_FrontLeg
- removed joint Torso_LeftLeg
- removed joint Torso_RightLeg
- added joint LeftLeg1_leftLowerLeg1: type revolute, parent LeftLeg1, child LeftLowerLeg1, origin xyz=0 -1 0 rpy=0 0 0, axis 0 1 0, limit lower=-3.14159 upper=3.14159 effort=0.0 velocity=0.0
- added joint LeftLeg3_LeftLowerLeg3: type revolute, parent LeftLeg3, child LeftLowerLeg3, origin xyz=0 -1 0 rpy=0 0 0, axis 0 1 0, limit lower=-3.14159 upper=3.14159 effort=0.0 velocity=0.0
- added joint RightLeg1_RightLowerLeg1: type revolute, parent Leg, child FrontLowerLeg, origin xyz=0 1 0 rpy=0 0 0, axis 0 1 0, limit lower=-3.14159 upper=3.14159 effort=0.0 velocity=0.0
- added joint RightLeg3_RightLowerLeg3: type revolute, parent RightLeg3, child RightLowerLeg3, origin xyz=0 1 0 rpy=0 0 0, axis 0 1 0, limit lower=-3.14159 upper=3.14159 effort=0.0 velocity=0.0
- added joint Torso_LeftLeg1: type revolute, parent Torso, child leftLeg1, origin xyz=-0.6 -0.5 3 rpy=0 0 0, axis 0 0 1, limit lower=-3.14159 upper=3.14159 effort=0.0 velocity=0.0
- added joint Torso_LeftLeg3: type revolute, parent Torso, child LeftLeg3, origin xyz=0.6 -0.5 3 rpy=0 0 0, axis 1 0 0, limit lower=-3.14159 upper=3.14159 effort=0.0 velocity=0.0
- added joint Torso_RightLeg1: type revolute, parent Torso, child RightLeg1, origin xyz=-0.6 0.5 3 rpy=0 0 0, axis 0 0 1, limit lower=-3.14159 upper=3.14159 effort=0.0 velocity=0.0
- added joint Torso_RightLeg3: type revolute, parent Torso, child RightLeg3, origin xyz=0.6 0.5 3 rpy=0 0 0, axis 1 0 0, limit lower=-3.14159 upper=3.14159 effort=0.0 velocity=0.0

Commit message: have a issue of keyerror

File: body.urdf (robot description, URDF)
Before this commit: robot robot, 9 links, 8 joints
Links:
- added link LeftLeg2, mass 1; collision box size=0.2 1 0.2; visual box size=0.2 1 0.2
- added link LeftLowerLeg2, mass 1; collision box size=0.2 0.2 1; visual box size=0.2 0.2 1
- added link RightLeg2, mass 1; collision box size=0.2 1 0.2; visual box size=0.2 1 0.2
- added link RightLowerLeg2, mass 1; collision box size=0.2 0.2 1; visual box size=0.2 0.2 1
Joints:
- added joint LeftLeg2_LeftLowerLeg2: type revolute, parent LeftLeg2, child LeftLowerLeg2, origin xyz=0 -1 0 rpy=0 0 0, axis 0 1 0, limit lower=-3.14159 upper=3.14159 effort=0.0 velocity=0.0
- added joint RightLeg2_RightLowerLeg2: type revolute, parent RightLeg2, child RightLowerLeg2, origin xyz=0 1 0 rpy=0 0 0, axis 0 1 0, limit lower=-3.14159 upper=3.14159 effort=0.0 velocity=0.0
- added joint Torso_LeftLeg2: type revolute, parent Torso, child LeftLeg2, origin xyz=0 -0.5 3 rpy=0 0 0, axis 0 0 1, limit lower=-3.14159 upper=3.14159 effort=0.0 velocity=0.0
- added joint Torso_RightLeg2: type revolute, parent Torso, child RightLeg2, origin xyz=0 0.5 3 rpy=0 0 0, axis 0 0 1, limit lower=-3.14159 upper=3.14159 effort=0.0 velocity=0.0
- joint RightLeg1_RightLowerLeg1: child FrontLowerLeg -> RightLowerLeg1; parent Leg -> RightLeg1
- joint Torso_LeftLeg1: child leftLeg1 -> LeftLeg1

Commit message: fix keyerror

File: body.urdf (robot description, URDF)
Before this commit: robot robot, 13 links, 12 joints
Joints:
- removed joint LeftLeg1_leftLowerLeg1
- added joint LeftLeg1_LeftLowerLeg1: type revolute, parent LeftLeg1, child LeftLowerLeg1, origin xyz=0 -1 0 rpy=0 0 0, axis 0 1 0, limit lower=-3.14159 upper=3.14159 effort=0.0 velocity=0.0

Commit message: creare a hexaped

File: body.urdf (robot description, URDF)
Before this commit: robot robot, 13 links, 12 joints
Joints:
- joint LeftLeg2_LeftLowerLeg2: axis 0 1 0 -> 1 0 0
- joint RightLeg2_RightLowerLeg2: axis 0 1 0 -> 1 0 0
- joint Torso_LeftLeg1: origin xyz=-0.6 -0.5 3 rpy=0 0 0 -> xyz=-1 -0.5 3 rpy=0 0 0
- joint Torso_LeftLeg2: axis 0 0 1 -> 1 0 0 
- joint Torso_LeftLeg3: axis 1 0 0 -> 0 0 1; origin xyz=0.6 -0.5 3 rpy=0 0 0 -> xyz=1 -0.5 3 rpy=0 0 0
- joint Torso_RightLeg1: origin xyz=-0.6 0.5 3 rpy=0 0 0 -> xyz=-1 0.5 3 rpy=0 0 0
- joint Torso_RightLeg2: axis 0 0 1 -> 1 0 0
- joint Torso_RightLeg3: axis 1 0 0 -> 0 0 1; origin xyz=0.6 0.5 3 rpy=0 0 0 -> xyz=1 0.5 3 rpy=0 0 0

Commit message: make four leg robot

File: body.urdf (robot description, URDF)
Before this commit: robot robot, 13 links, 12 joints
Links:
- removed link LeftLeg3
- removed link LeftLowerLeg3
- removed link RightLeg3
- removed link RightLowerLeg3
- link Torso: geometry collision box size=1 1 1; visual box size=1 1 1
Joints:
- removed joint LeftLeg3_LeftLowerLeg3
- removed joint RightLeg3_RightLowerLeg3
- removed joint Torso_LeftLeg3
- removed joint Torso_RightLeg3
- joint Torso_LeftLeg1: origin xyz=-1 -0.5 3 rpy=0 0 0 -> xyz=-0.5 -0.5 2 rpy=0 0 0
- joint Torso_LeftLeg2: origin xyz=0 -0.5 3 rpy=0 0 0 -> xyz=0.5 -0.5 2 rpy=0 0 0
- joint Torso_RightLeg1: origin xyz=-1 0.5 3 rpy=0 0 0 -> xyz=-0.5 0.5 2 rpy=0 0 0
- joint Torso_RightLeg2: origin xyz=0 0.5 3 rpy=0 0 0 -> xyz=0.5 0.5 2 rpy=0 0 0

Commit message: make robot go down stairs

File: body.urdf (robot description, URDF)
Before this commit: robot robot, 9 links, 8 joints
Joints:
- joint Torso_LeftLeg1: origin xyz=-0.5 -0.5 2 rpy=0 0 0 -> xyz=-0.5 -0.5 5 rpy=0 0 0
- joint Torso_LeftLeg2: origin xyz=0.5 -0.5 2 rpy=0 0 0 -> xyz=0.5 -0.5 5 rpy=0 0 0
- joint Torso_RightLeg1: origin xyz=-0.5 0.5 2 rpy=0 0 0 -> xyz=-0.5 0.5 5 rpy=0 0 0
- joint Torso_RightLeg2: origin xyz=0.5 0.5 2 rpy=0 0 0 -> xyz=0.5 0.5 5 rpy=0 0 0

Commit message: finish walk down stairs

File: body.urdf (robot description, URDF)
Before this commit: robot robot, 9 links, 8 joints
Joints:
- joint Torso_LeftLeg1: origin xyz=-0.5 -0.5 5 rpy=0 0 0 -> xyz=-0.5 -0.5 3 rpy=0 0 0
- joint Torso_LeftLeg2: origin xyz=0.5 -0.5 5 rpy=0 0 0 -> xyz=0.5 -0.5 3 rpy=0 0 0
- joint Torso_RightLeg1: origin xyz=-0.5 0.5 5 rpy=0 0 0 -> xyz=-0.5 0.5 3 rpy=0 0 0
- joint Torso_RightLeg2: origin xyz=0.5 0.5 5 rpy=0 0 0 -> xyz=0.5 0.5 3 rpy=0 0 0

Commit message: Make a four leg bug that walk down stairs

File: body.urdf (robot description, URDF)
Before this commit: robot robot, 9 links, 8 joints
Links:
- removed link Torso
- added link Head, mass 1; collision box size=0.6 0.6 0.6; visual box size=0.6 0.6 0.6
- added link Torso1, mass 1; collision box size=1 1 1; visual box size=1 1 1
- added link Torso2, mass 1; collision box size=1.2 1.2 1.2; visual box size=1.2 1.2 1.2
Joints:
- removed joint Torso_LeftLeg1
- removed joint Torso_LeftLeg2
- removed joint Torso_RightLeg1
- removed joint Torso_RightLeg2
- added joint Torso1_Head: type revolute, parent Torso1, child Head, origin xyz=-0.5 0 3 rpy=0 0 0, axis 0 1 0, limit lower=-3.14159 upper=3.14159 effort=0.0 velocity=0.0
- added joint Torso1_LeftLeg1: type revolute, parent Torso1, child LeftLeg1, origin xyz=-0.2 -0.5 3 rpy=0 0 0, axis 0 0 1, limit lower=-3.14159 upper=3.14159 effort=0.0 velocity=0.0
- added joint Torso1_RightLeg1: type revolute, parent Torso1, child RightLeg1, origin xyz=-0.2 0.5 3 rpy=0 0 0, axis 0 0 1, limit lower=-3.14159 upper=3.14159 effort=0.0 velocity=0.0
- added joint Torso1_Torso2: type revolute, parent Torso1, child Torso2, origin xyz=0.5 0 3 rpy=0 0 0, axis 0 1 0, limit lower=-3.14159 upper=3.14159 effort=0.0 velocity=0.0
- added joint Torso2_LeftLeg2: type revolute, parent Torso2, child LeftLeg2, origin xyz=0.8 -0.5 0 rpy=0 0 0, axis 1 0 0, limit lower=-3.14159 upper=3.14159 effort=0.0 velocity=0.0
- added joint Torso2_RightLeg2: type revolute, parent Torso2, child RightLeg2, origin xyz=0.8 0.5 0 rpy=0 0 0, axis 1 0 0, limit lower=-3.14159 upper=3.14159 effort=0.0 velocity=0.0

Commit message: generate random bodies

File: body.urdf (robot description, URDF)
Before this commit: robot robot, 11 links, 10 joints
Links:
- removed link Head
- removed link LeftLeg1
- removed link LeftLeg2
- removed link LeftLowerLeg1
- removed link LeftLowerLeg2
- removed link RightLeg1
- removed link RightLeg2
- removed link RightLowerLeg1
- removed link RightLowerLeg2
- added link Torso3, mass 1; collision box size=0.8137278571279575 0.8838178291021835 0.8683323603899004; visual box size=0.8137278571279575 0.8838178291021835 0.8683323603899004
- added link Torso4, mass 1; collision box size=0.4899368100724598 0.45400185859945885 0.6132641790587987; visual box size=0.4899368100724598 0.45400185859945885 0.6132641790587987
- added link Torso5, mass 1; collision box size=0.7227338707120687 0.010167537454707887 0.9043427595181945; visual box size=0.7227338707120687 0.010167537454707887 0.9043427595181945
- added link Torso6, mass 1; collision box size=0.06149570045793906 0.576801161696996 0.23502888462227656; visual box size=0.06149570045793906 0.576801161696996 0.23502888462227656
- link Torso1: geometry collision box size=0.1508909230678307 0.20798078580769497 0.8484272564035092; visual box size=0.1508909230678307 0.20798078580769497 0.8484272564035092
- link Torso2: geometry collision box size=0.28726861095615275 0.43229124969720545 0.8722880486512228; visual box size=0.28726861095615275 0.43229124969720545 0.8722880486512228
Joints:
- removed joint LeftLeg1_LeftLowerLeg1
- removed joint LeftLeg2_LeftLowerLeg2
- removed joint RightLeg1_RightLowerLeg1
- removed joint RightLeg2_RightLowerLeg2
- removed joint Torso1_Head
- removed joint Torso1_LeftLeg1
- removed joint Torso1_RightLeg1
- removed joint Torso2_LeftLeg2
- removed joint Torso2_RightLeg2
- added joint Torso02_Torso3: type revolute, parent Torso2, child Torso3, origin xyz=0.28726861095615275 0 0 rpy=0 0 0, axis 0 1 0, limit lower=-3.14159 upper=3.14159 effort=0.0 velocity=0.0
- added joint Torso03_Torso4: type revolute, parent Torso3, child Torso4, origin xyz=0.8137278571279575 0 0 rpy=0 0 0, axis 0 1 0, limit lower=-3.14159 upper=3.14159 effort=0.0 velocity=0.0
- added joint Torso04_Torso5: type revolute, parent Torso4, child Torso5, origin xyz=0.4899368100724598 0 0 rpy=0 0 0, axis 0 1 0, limit lower=-3.14159 upper=3.14159 effort=0.0 velocity=0.0
- added joint Torso05_Torso6: type revolute, parent Torso5, child Torso6, origin xyz=0.7227338707120687 0 0 rpy=0 0 0, axis 0 1 0, limit lower=-3.14159 upper=3.14159 effort=0.0 velocity=0.0
- joint Torso1_Torso2: origin xyz=0.5 0 3 rpy=0 0 0 -> xyz=0.07544546153391535 0 3 rpy=0 0 0

Commit message: finish generate 1D snake

File: body.urdf (robot description, URDF)
Before this commit: robot robot, 6 links, 5 joints
Links:
- added link Torso10, mass 1; collision box size=0.8649306556441176 0.9084130209439196 0.8746887639746598; visual box size=0.8649306556441176 0.9084130209439196 0.8746887639746598
- added link Torso7, mass 1; collision box size=0.38627928528376665 0.356955352087743 0.21497833211072048; visual box size=0.38627928528376665 0.356955352087743 0.21497833211072048
- added link Torso8, mass 1; collision box size=0.6093151580227867 0.11743816471765045 0.7234943856587951; visual box size=0.6093151580227867 0.11743816471765045 0.7234943856587951
- added link Torso9, mass 1; collision box size=0.02327440239771994 0.0812156421512702 0.8625370461338405; visual box size=0.02327440239771994 0.0812156421512702 0.8625370461338405
- link Torso1: geometry collision box size=0.8120906944912345 0.35010568889953053 0.4785435973101613; visual box size=0.8120906944912345 0.35010568889953053 0.4785435973101613
- link Torso2: geometry collision box size=0.9462745129646449 0.28251851796759564 0.3903095950873555; visual box size=0.9462745129646449 0.28251851796759564 0.3903095950873555
- link Torso3: geometry collision box size=0.07523186244251356 0.15153419753810482 0.5670925991490906; visual box size=0.07523186244251356 0.15153419753810482 0.5670925991490906
- link Torso4: geometry collision box size=0.23212717967154195 0.06906175693854433 0.6984504197447119; visual box size=0.23212717967154195 0.06906175693854433 0.6984504197447119
- link Torso5: geometry collision box size=0.1334031676790408 0.9144861625037822 0.2705282937929485; visual box size=0.1334031676790408 0.9144861625037822 0.2705282937929485
- link Torso6: geometry collision box size=0.2715350290887395 0.6301709185730674 0.6614290641003125; visual box size=0.2715350290887395 0.6301709185730674 0.6614290641003125
Joints:
- removed joint Torso02_Torso3
- removed joint Torso03_Torso4
- removed joint Torso04_Torso5
- removed joint Torso05_Torso6
- added joint Torso2_Torso3: type revolute, parent Torso2, child Torso3, origin xyz=0.9462745129646449 0 0 rpy=0 0 0, axis 0 1 0, limit lower=-3.14159 upper=3.14159 effort=0.0 velocity=0.0
- added joint Torso3_Torso4: type revolute, parent Torso3, child Torso4, origin xyz=0.07523186244251356 0 0 rpy=0 0 0, axis 0 1 0, limit lower=-3.14159 upper=3.14159 effort=0.0 velocity=0.0
- added joint Torso4_Torso5: type revolute, parent Torso4, child Torso5, origin xyz=0.23212717967154195 0 0 rpy=0 0 0, axis 0 1 0, limit lower=-3.14159 upper=3.14159 effort=0.0 velocity=0.0
- added joint Torso5_Torso6: type revolute, parent Torso5, child Torso6, origin xyz=0.1334031676790408 0 0 rpy=0 0 0, axis 0 1 0, limit lower=-3.14159 upper=3.14159 effort=0.0 velocity=0.0
- added joint Torso6_Torso7: type revolute, parent Torso6, child Torso7, origin xyz=0.2715350290887395 0 0 rpy=0 0 0, axis 0 1 0, limit lower=-3.14159 upper=3.14159 effort=0.0 velocity=0.0
- added joint Torso7_Torso8: type revolute, parent Torso7, child Torso8, origin xyz=0.38627928528376665 0 0 rpy=0 0 0, axis 0 1 0, limit lower=-3.14159 upper=3.14159 effort=0.0 velocity=0.0
- added joint Torso8_Torso9: type revolute, parent Torso8, child Torso9, origin xyz=0.6093151580227867 0 0 rpy=0 0 0, axis 0 1 0, limit lower=-3.14159 upper=3.14159 effort=0.0 velocity=0.0
- added joint Torso9_Torso10: type revolute, parent Torso9, child Torso10, origin xyz=0.02327440239771994 0 0 rpy=0 0 0, axis 0 1 0, limit lower=-3.14159 upper=3.14159 effort=0.0 velocity=0.0
- joint Torso1_Torso2: origin xyz=0.07544546153391535 0 3 rpy=0 0 0 -> xyz=0.40604534724561725 0 3 rpy=0 0 0

Commit message: do one generation of 1-D snake at a time

File: body.urdf (robot description, URDF)
Before this commit: robot robot, 10 links, 9 joints
Links:
- removed link Torso10
- removed link Torso8
- removed link Torso9
- link Torso1: geometry collision box size=0.9192819226884376 0.35944584015082637 0.42713123121768193; visual box size=0.9192819226884376 0.35944584015082637 0.42713123121768193
- link Torso2: geometry collision box size=0.37182262104980845 0.010273825992943908 0.13131403102753447; visual box size=0.37182262104980845 0.010273825992943908 0.13131403102753447
- link Torso3: geometry collision box size=0.8075406676853192 0.01455062744509128 0.48781756768330586; visual box size=0.8075406676853192 0.01455062744509128 0.48781756768330586
- link Torso4: geometry collision box size=0.4135925012873355 0.6023879569009531 0.8982193001042452; visual box size=0.4135925012873355 0.6023879569009531 0.8982193001042452
- link Torso5: geometry collision box size=0.081184455645816 0.6853533074941169 0.5199613112598941; visual box size=0.081184455645816 0.6853533074941169 0.5199613112598941
- link Torso6: geometry collision box size=0.24401166075874903 0.7992384305393121 0.7502561711703372; visual box size=0.24401166075874903 0.7992384305393121 0.7502561711703372
- link Torso7: geometry collision box size=0.86265622642153 0.6108707812268714 0.14632996609405013; visual box size=0.86265622642153 0.6108707812268714 0.14632996609405013
Joints:
- removed joint Torso7_Torso8
- removed joint Torso8_Torso9
- removed joint Torso9_Torso10
- joint Torso1_Torso2: origin xyz=0.40604534724561725 0 3 rpy=0 0 0 -> xyz=0.4596409613442188 0 2 rpy=0 0 0
- joint Torso2_Torso3: origin xyz=0.9462745129646449 0 0 rpy=0 0 0 -> xyz=0.37182262104980845 0 0 rpy=0 0 0
- joint Torso3_Torso4: origin xyz=0.07523186244251356 0 0 rpy=0 0 0 -> xyz=0.8075406676853192 0 0 rpy=0 0 0
- joint Torso4_Torso5: origin xyz=0.23212717967154195 0 0 rpy=0 0 0 -> xyz=0.4135925012873355 0 0 rpy=0 0 0
- joint Torso5_Torso6: origin xyz=0.1334031676790408 0 0 rpy=0 0 0 -> xyz=0.081184455645816 0 0 rpy=0 0 0
- joint Torso6_Torso7: origin xyz=0.2715350290887395 0 0 rpy=0 0 0 -> xyz=0.24401166075874903 0 0 rpy=0 0 0
