Commit message: debugging repeated link name

File: body.urdf (robot description, URDF)
Before this commit: robot robot, 7 links, 6 joints
Links:
- added link Torso0, mass 1; collision box size=0.9834299016898991 0.9535418122166881 0.9884933254562791; visual box size=0.9834299016898991 0.9535418122166881 0.9884933254562791
- added link Torso8, mass 1; collision box size=0.70420138842031 0.5144102456611759 0.9624256335291683; visual box size=0.70420138842031 0.5144102456611759 0.9624256335291683
- added link Torso9, mass 1; collision box size=0.25832080730400037 0.5502978698105236 0.9506285388553133; visual box size=0.25832080730400037 0.5502978698105236 0.9506285388553133
- link Torso1: geometry collision box size=0.8773263886688192 0.9797878092431884 0.7401776171317087; visual box size=0.8773263886688192 0.9797878092431884 0.7401776171317087
- link Torso2: geometry collision box size=0.5197652186529372 0.2613874724387819 0.9093074072096348; visual box size=0.5197652186529372 0.2613874724387819 0.9093074072096348
- link Torso3: geometry collision box size=0.6896027099604989 0.37445240797361556 0.8154905168809945; visual box size=0.6896027099604989 0.37445240797361556 0.8154905168809945
- link Torso4: geometry collision box size=0.45748683440173754 0.8767437755305698 0.5602042456433074; visual box size=0.45748683440173754 0.8767437755305698 0.5602042456433074
- link Torso5: geometry collision box size=0.6695032769341137 0.6865550388647688 0.7471768969134132; visual box size=0.6695032769341137 0.6865550388647688 0.7471768969134132
- link Torso6: geometry collision box size=0.788074801397395 0.9539419329987648 0.48914708838390164; visual box size=0.788074801397395 0.9539419329987648 0.48914708838390164
- link Torso7: geometry collision box size=0.444110944971869 0.5146078777490293 0.9198353915582449; visual box size=0.444110944971869 0.5146078777490293 0.9198353915582449
Joints:
- added joint Torso0_Torso1: type revolute, parent Torso0, child Torso1, origin xyz=0.49171495084494954 0 1 rpy=0 0 0, axis 0 0 1, limit lower=-3.14159 upper=3.14159 effort=0.0 velocity=0.0
- added joint Torso7_Torso8: type revolute, parent Torso7, child Torso8, origin xyz=0.2220554724859345 0 0.45991769577912245 rpy=0 0 0, axis 1 0 0, limit lower=-3.14159 upper=3.14159 effort=0.0 velocity=0.0
- added joint Torso8_Torso9: type revolute, parent Torso8, child Torso9, origin xyz=0 0.25720512283058794 0.48121281676458416 rpy=0 0 0, axis 1 0 0, limit lower=-3.14159 upper=3.14159 effort=0.0 velocity=0.0
- joint Torso1_Torso2: axis 0 1 0 -> 1 0 0; origin xyz=0.4596409613442188 0 2 rpy=0 0 0 -> xyz=0.4386631943344096 0.4898939046215942 0 rpy=0 0 0
- joint Torso2_Torso3: axis 0 1 0 -> 1 0 0; origin xyz=0.37182262104980845 0 0 rpy=0 0 0 -> xyz=0 0.13069373621939095 0.4546537036048174 rpy=0 0 0
- joint Torso3_Torso4: axis 0 1 0 -> 1 0 0; origin xyz=0.8075406676853192 0 0 rpy=0 0 0 -> xyz=0.34480135498024944 0 0.40774525844049725 rpy=0 0 0
- joint Torso4_Torso5: axis 0 1 0 -> 1 0 0; origin xyz=0.4135925012873355 0 0 rpy=0 0 0 -> xyz=0.22874341720086877 0 0.2801021228216537 rpy=0 0 0
- joint Torso5_Torso6: axis 0 1 0 -> 1 0 0; origin xyz=0.081184455645816 0 0 rpy=0 0 0 -> xyz=0 0.3432775194323844 0.3735884484567066 rpy=0 0 0
- joint Torso6_Torso7: axis 0 1 0 -> 1 0 0; origin xyz=0.24401166075874903 0 0 rpy=0 0 0 -> xyz=0.3940374006986975 0.4769709664993824 0 rpy=0 0 0

File: body0.urdf (robot description, URDF)
Before this commit: robot robot, 9 links, 8 joints
Links:
- removed link Torso6
- removed link Torso7
- removed link Torso8
- link Torso0: geometry collision box size=0.7221266454020552 0.4258501196434774 0.4473223048255787; visual box size=0.7221266454020552 0.4258501196434774 0.4473223048255787
- link Torso1: geometry collision box size=0.9628286295986108 0.7384400451068263 0.7709084048256509; visual box size=0.9628286295986108 0.7384400451068263 0.7709084048256509
- link Torso2: geometry collision box size=0.4327980652241805 0.4755243051272151 0.7766051976000437; visual box size=0.4327980652241805 0.4755243051272151 0.7766051976000437
- link Torso3: geometry collision box size=0.6352962473612347 0.47391765394449376 0.8856941809444161; visual box size=0.6352962473612347 0.47391765394449376 0.8856941809444161
- link Torso4: geometry collision box size=0.7285388303274021 0.335549106058989 0.9022440389529256; visual box size=0.7285388303274021 0.335549106058989 0.9022440389529256
- link Torso5: geometry collision box size=0.6714890490356322 0.7351964194609808 0.28838689269340484; visual box size=0.6714890490356322 0.7351964194609808 0.28838689269340484
Joints:
- removed joint Torso5_Torso6
- removed joint Torso6_Torso7
- removed joint Torso7_Torso8
- joint Torso0_Torso1: origin xyz=0.30923034956830053 0 1 rpy=0 0 0 -> xyz=0.3610633227010276 0 1 rpy=0 0 0; parent Torso8 -> Torso5
- joint Torso1_Torso2: axis 0 1 0 -> 0 0 1; origin xyz=0.33864713386682377 0.3653320329558286 0 rpy=0 0 0 -> xyz=0.21292542224677075 0.11606071077364787 0 rpy=0 0 0
- joint Torso2_Torso3: axis 0 1 0 -> 0 0 1; origin xyz=0.48775516053954804 0 0.36457428699478234 rpy=0 0 0 -> xyz=0.40434474700711887 0.16930167865884826 0 rpy=0 0 0
- joint Torso3_Torso4: origin xyz=0.17826178434508258 0.2056884250561638 0 rpy=0 0 0 -> xyz=0.31827613670805077 0.2993988362918181 0 rpy=0 0 0
- joint Torso4_Torso5: axis 1 0 0 -> 0 1 0; child Torso4 -> Torso5; origin xyz=0.49034370390739024 0.4787699038810528 0 rpy=0 0 0 -> xyz=0.2909702646593355 0 0.4710905364155259 rpy=0 0 0; parent Torso3 -> Torso4
