Commit message: update README

File: body0.urdf (robot description, URDF)
Before this commit: robot robot, 9 links, 8 joints
Links:
- removed link Torso3
- removed link Torso4
- removed link Torso5
- removed link Torso6
- removed link Torso7
- removed link Torso8
- removed link Torso9
- link Torso1: geometry collision box size=0.09360974642781572 0.6697014306381986 0.15012744005170564; visual box size=0.09360974642781572 0.6697014306381986 0.15012744005170564
- link Torso2: geometry collision box size=0.2675736632733723 0.8170870459537963 0.6080286473243297; visual box size=0.2675736632733723 0.8170870459537963 0.6080286473243297
Joints:
- removed joint Torso2_Torso3
- removed joint Torso3_Torso4
- removed joint Torso4_Torso5
- removed joint Torso5_Torso6
- removed joint Torso6_Torso7
- removed joint Torso7_Torso8
- removed joint Torso8_Torso9
- joint Torso1_Torso2: origin xyz=0.3944107600549284 0 2 rpy=0 0 0 -> xyz=0.04680487321390786 0 2 rpy=0 0 0

Commit message: disable sidebar when simulate

File: body0.urdf (robot description, URDF)
Before this commit: robot robot, 2 links, 1 joints
Links:
- added link Torso3, mass 1; collision box size=0.03985466922880765 0.7238851133334331 0.6769890860384591; visual box size=0.03985466922880765 0.7238851133334331 0.6769890860384591
- added link Torso4, mass 1; collision box size=0.5756461901861486 0.717297825726533 0.2688880147871111; visual box size=0.5756461901861486 0.717297825726533 0.2688880147871111
- link Torso1: geometry collision box size=0.8783866279963414 0.9702512706364166 0.8692500897019005; visual box size=0.8783866279963414 0.9702512706364166 0.8692500897019005
- link Torso2: geometry collision box size=0.15911818504159636 0.719428718122882 0.26163895515815894; visual box size=0.15911818504159636 0.719428718122882 0.26163895515815894
Joints:
- added joint Torso2_Torso3: type revolute, parent Torso2, child Torso3, origin xyz=0.15911818504159636 0 0 rpy=0 0 0, axis 0 1 0, limit lower=-3.14159 upper=3.14159 effort=0.0 velocity=0.0
- added joint Torso3_Torso4: type revolute, parent Torso3, child Torso4, origin xyz=0.03985466922880765 0 0 rpy=0 0 0, axis 0 1 0, limit lower=-3.14159 upper=3.14159 effort=0.0 velocity=0.0
- joint Torso1_Torso2: origin xyz=0.04680487321390786 0 2 rpy=0 0 0 -> xyz=0.4391933139981707 0 2 rpy=0 0 0

Commit message: create 3D snake

File: body0.urdf (robot description, URDF)
Before this commit: robot robot, 4 links, 3 joints
Links:
- added link Torso0, mass 1; collision box size=0.6184606991366011 0.9344666434625342 0.4836424808869751; visual box size=0.6184606991366011 0.9344666434625342 0.4836424808869751
- added link Torso5, mass 1; collision box size=0.7642456568113443 0.4373625841149011 0.91898536819472; visual box size=0.7642456568113443 0.4373625841149011 0.91898536819472
- added link Torso6, mass 1; collision box size=0.836095050163481 0.5007150011888071 0.5857603387275698; visual box size=0.836095050163481 0.5007150011888071 0.5857603387275698
- added link Torso7, mass 1; collision box size=0.9456802497455372 0.7857935757706098 0.7396133723095908; visual box size=0.9456802497455372 0.7857935757706098 0.7396133723095908
- added link Torso8, mass 1; collision box size=0.9376685668059339 0.9152174567829692 0.7174525160392808; visual box size=0.9376685668059339 0.9152174567829692 0.7174525160392808
- link Torso1: geometry collision box size=0.919678873742815 0.3016290322368305 0.6235629040653722; visual box size=0.919678873742815 0.3016290322368305 0.6235629040653722
- link Torso2: geometry collision box size=0.3209738738056991 0.5234004395270755 0.7063937157097551; visual box size=0.3209738738056991 0.5234004395270755 0.7063937157097551
- link Torso3: geometry collision box size=0.7952227773901563 0.7440701043829965 0.3850512871323064; visual box size=0.7952227773901563 0.7440701043829965 0.3850512871323064
- link Torso4: geometry collision box size=0.4989504441570194 0.37711856175305813 0.9404673298882265; visual box size=0.4989504441570194 0.37711856175305813 0.9404673298882265
Joints:
- added joint Torso0_Torso1: type revolute, parent Torso8, child Torso0, origin xyz=0.30923034956830053 0 1 rpy=0 0 0, axis 0 1 0, limit lower=-3.14159 upper=3.14159 effort=0.0 velocity=0.0
- added joint Torso4_Torso5: type revolute, parent Torso3, child Torso4, origin xyz=0.49034370390739024 0.4787699038810528 0 rpy=0 0 0, axis 1 0 0, limit lower=-3.14159 upper=3.14159 effort=0.0 velocity=0.0
- added joint Torso5_Torso6: type revolute, parent Torso4, child Torso5, origin xyz=0.3222141042842369 0.4020078068905464 0 rpy=0 0 0, axis 0 0 1, limit lower=-3.14159 upper=3.14159 effort=0.0 velocity=0.0
- added joint Torso6_Torso7: type revolute, parent Torso5, child Torso6, origin xyz=0 0.3397836202834018 0.4354502463519708 rpy=0 0 0, axis 0 0 1, limit lower=-3.14159 upper=3.14159 effort=0.0 velocity=0.0
- added joint Torso7_Torso8: type revolute, parent Torso6, child Torso7, origin xyz=0.36711237252132467 0.330485197341681 0 rpy=0 0 0, axis 0 0 1, limit lower=-3.14159 upper=3.14159 effort=0.0 velocity=0.0
- joint Torso1_Torso2: child Torso2 -> Torso1; origin xyz=0.4391933139981707 0 2 rpy=0 0 0 -> xyz=0.33864713386682377 0.3653320329558286 0 rpy=0 0 0; parent Torso1 -> Torso0
- joint Torso2_Torso3: child Torso3 -> Torso2; origin xyz=0.15911818504159636 0 0 rpy=0 0 0 -> xyz=0.48775516053954804 0 0.36457428699478234 rpy=0 0 0; parent Torso2 -> Torso1
- joint Torso3_Torso4: axis 0 1 0 -> 1 0 0; child Torso4 -> Torso3; origin xyz=0.03985466922880765 0 0 rpy=0 0 0 -> xyz=0.17826178434508258 0.2056884250561638 0 rpy=0 0 0; parent Torso3 -> Torso2

Commit message: first link stuck in ground

File: body0.urdf (robot description, URDF)
Before this commit: robot robot, 6 links, 5 joints
Links:
- removed link Torso0
- link Torso1: geometry collision box size=0.2924475531447507 0.6649622807900465 0.952278840755999; visual box size=0.2924475531447507 0.6649622807900465 0.952278840755999
- link Torso2: geometry collision box size=0.4665122347353746 0.526150155365436 0.6938396056281617; visual box size=0.4665122347353746 0.526150155365436 0.6938396056281617
- link Torso3: geometry collision box size=0.3759739922076179 0.6317831267863729 0.5213139022658826; visual box size=0.3759739922076179 0.6317831267863729 0.5213139022658826
- link Torso4: geometry collision box size=0.9276986049309723 0.7587466254676687 0.4096115700056472; visual box size=0.9276986049309723 0.7587466254676687 0.4096115700056472
- link Torso5: geometry collision box size=0.790836107560984 0.8552240746934092 0.7047249744621065; visual box size=0.790836107560984 0.8552240746934092 0.7047249744621065
Joints:
- removed joint Torso0_Torso1
- joint Torso1_Torso2: axis 0 0 1 -> 0 1 0; child Torso1 -> Torso2; origin xyz=0.21292542224677075 0.11606071077364787 0 rpy=0 0 0 -> xyz=0.14622377657237534 0.33248114039502324 0 rpy=0 0 0; parent Torso0 -> Torso1
- joint Torso2_Torso3: axis 0 0 1 -> 0 1 0; child Torso2 -> Torso3; origin xyz=0.40434474700711887 0.16930167865884826 0 rpy=0 0 0 -> xyz=0.2332561173676873 0 0.34691980281408086 rpy=0 0 0; parent Torso1 -> Torso2
- joint Torso3_Torso4: child Torso3 -> Torso4; origin xyz=0.31827613670805077 0.2993988362918181 0 rpy=0 0 0 -> xyz=0.18798699610380895 0 0.2606569511329413 rpy=0 0 0; parent Torso2 -> Torso3
- joint Torso4_Torso5: axis 0 1 0 -> 1 0 0; origin xyz=0.2909702646593355 0 0.4710905364155259 rpy=0 0 0 -> xyz=0.46384930246548617 0 0.2048057850028236 rpy=0 0 0
